Commit message: Set the perspective projection for projective texture mapping. Change the demo to two bears with the same view projection matrix for the camera and the projector.

File: data/teddy_large.urdf (robot description, URDF)
Before this commit: robot cube.urdf, 1 links, 0 joints
Links:
- link baseLink: geometry collision mesh filename=teddy2_VHACD_CHs.obj scale=3 3 3; visual mesh filename=teddy2_VHACD_CHs.obj scale=3 3 3
